Commit message: Lappa v0.2: multi ROS2 distro, package bundler, 3D mesh attach
- Select humble/iron/jazzy/kilted/rolling; rewrite Dockerfiles for Docker show
- Bundle ROS2 packages into colcon-ready zip with lappa_manifest.json
- Procedural OBJ meshes (chassis/wheel/arm/lidar) attach into package URDF
- IDE: ROS2 dropdown, Package panel, Models panel; CLI + API + tests

File: packages/demos/diff_drive_2w/urdf/robot.urdf (robot description, URDF)
Before this commit: robot diff_drive_2w, 3 links, 0 joints
Links:
- added link base_link_mesh; collision mesh filename=package://diff_drive_2w/meshes/unit_wheel.obj scale=1 1 1; visual mesh filename=package://diff_drive_2w/meshes/unit_wheel.obj scale=1 1 1
- link base_link: geometry collision mesh filename=package://diff_drive_2w/meshes/unit_wheel.obj scale=1 1 1; visual mesh filename=package://diff_drive_2w/meshes/unit_wheel.obj scale=1 1 1

File: packages/demos/omni_3w/urdf/robot.urdf (robot description, URDF)
Before this commit: robot omni_3w, 3 links, 0 joints
Links:
- added link base_link_mesh; collision mesh filename=package://omni_3w/meshes/api_chassis.obj scale=1 1 1; visual mesh filename=package://omni_3w/meshes/api_chassis.obj scale=1 1 1
- link base_link: geometry collision mesh filename=package://omni_3w/meshes/api_chassis.obj scale=1 1 1; visual mesh filename=package://omni_3w/meshes/api_chassis.obj scale=1 1 1

Commit message: Improve Lappa: export sim trajectory as CSV
- Session records odom trail; CLI sim trajectory and GET /api/sim/trajectory.csv
- Demo writes demo_trajectory.csv; bump 0.2.2

File: packages/demos/diff_drive_2w/urdf/robot.urdf (robot description, URDF)
Before this commit: robot diff_drive_2w, 4 links, 0 joints
Links:
- link base_link_mesh: geometry collision mesh filename=package://diff_drive_2w/meshes/demo_chassis.obj scale=1 1 1; visual mesh filename=package://diff_drive_2w/meshes/demo_chassis.obj scale=1 1 1
