Commit message: feat(3d): full mesh fit, aligned multi-link robots, WebGL viewer
Auto-fit OBJ AABB to link size, build chassis+wheels+lidar with kinematic offsets and continuous joints, scene3d API, IDE 2D/3D toggle with Three.js orbit, sanitize legacy URDF spam. Bump to 0.3.0.

File: packages/demos/ackermann_4w/urdf/robot.urdf (robot description, URDF)
Before this commit: robot ackermann_4w, 3 links, 0 joints
Links:
- removed link wheel_left
- removed link wheel_right
- added link base_footprint
- added link lidar_link; collision mesh filename=package://ackermann_4w/meshes/ackermann_4w_lidar.obj scale=1 1 1; visual mesh filename=package://ackermann_4w/meshes/ackermann_4w_lidar.obj scale=1 1 1
- added link wheel_fl; collision mesh filename=package://ackermann_4w/meshes/ackermann_4w_wheel_fl.obj scale=1 1 1; visual mesh filename=package://ackermann_4w/meshes/ackermann_4w_wheel_fl.obj scale=1 1 1
- added link wheel_fr; collision mesh filename=package://ackermann_4w/meshes/ackermann_4w_wheel_fr.obj scale=1 1 1; visual mesh filename=package://ackermann_4w/meshes/ackermann_4w_wheel_fr.obj scale=1 1 1
- added link wheel_rl; collision mesh filename=package://ackermann_4w/meshes/ackermann_4w_wheel_rl.obj scale=1 1 1; visual mesh filename=package://ackermann_4w/meshes/ackermann_4w_wheel_rl.obj scale=1 1 1
- added link wheel_rr; collision mesh filename=package://ackermann_4w/meshes/ackermann_4w_wheel_rr.obj scale=1 1 1; visual mesh filename=package://ackermann_4w/meshes/ackermann_4w_wheel_rr.obj scale=1 1 1
- link base_link: geometry collision mesh filename=package://ackermann_4w/meshes/ackermann_4w_chassis.obj scale=1 1 1; visual mesh filename=package://ackermann_4w/meshes/ackermann_4w_chassis.obj scale=1 1 1
Joints:
- added joint base_joint: type fixed, parent base_footprint, child base_link, origin xyz=0 0 0.09000 rpy=0 0 0
- added joint lidar_joint: type fixed, parent base_link, child lidar_link, origin xyz=0.10000 0.00000 0.09000 rpy=0 0 0
- added joint wheel_fl_joint: type continuous, parent base_link, child wheel_fl, origin xyz=0.18000 0.14000 -0.04000 rpy=0 0 0.00000, axis 0 1 0
- added joint wheel_fr_joint: type continuous, parent base_link, child wheel_fr, origin xyz=0.18000 -0.14000 -0.04000 rpy=0 0 0.00000, axis 0 1 0
- added joint wheel_rl_joint: type continuous, parent base_link, child wheel_rl, origin xyz=-0.18000 0.14000 -0.04000 rpy=0 0 0.00000, axis 0 1 0
- added joint wheel_rr_joint: type continuous, parent base_link, child wheel_rr, origin xyz=-0.18000 -0.14000 -0.04000 rpy=0 0 0.00000, axis 0 1 0

File: packages/demos/diff_drive_2w/urdf/robot.urdf (robot description, URDF)
Before this commit: robot diff_drive_2w, 4 links, 0 joints
Links:
- removed link base_link_mesh
- added link base_footprint
- added link lidar_link; collision mesh filename=package://diff_drive_2w/meshes/diff_drive_2w_lidar.obj scale=1 1 1; visual mesh filename=package://diff_drive_2w/meshes/diff_drive_2w_lidar.obj scale=1 1 1
- link base_link: geometry collision mesh filename=package://diff_drive_2w/meshes/diff_drive_2w_chassis.obj scale=1 1 1; visual mesh filename=package://diff_drive_2w/meshes/diff_drive_2w_chassis.obj scale=1 1 1
- link wheel_left: geometry collision mesh filename=package://diff_drive_2w/meshes/diff_drive_2w_wheel_left.obj scale=1 1 1; visual mesh filename=package://diff_drive_2w/meshes/diff_drive_2w_wheel_left.obj scale=1 1 1
- link wheel_right: geometry collision mesh filename=package://diff_drive_2w/meshes/diff_drive_2w_wheel_right.obj scale=1 1 1; visual mesh filename=package://diff_drive_2w/meshes/diff_drive_2w_wheel_right.obj scale=1 1 1
Joints:
- added joint base_joint: type fixed, parent base_footprint, child base_link, origin xyz=0 0 0.08000 rpy=0 0 0
- added joint lidar_joint: type fixed, parent base_link, child lidar_link, origin xyz=0.05000 0.00000 0.08000 rpy=0 0 0
- added joint wheel_left_joint: type continuous, parent base_link, child wheel_left, origin xyz=0.00000 0.16000 -0.03000 rpy=0 0 0.00000, axis 0 1 0
- added joint wheel_right_joint: type continuous, parent base_link, child wheel_right, origin xyz=0.00000 -0.16000 -0.03000 rpy=0 0 0.00000, axis 0 1 0

File: packages/demos/omni_3w/urdf/robot.urdf (robot description, URDF)
Before this commit: robot omni_3w, 4 links, 0 joints
Links:
- removed link base_link_mesh
- removed link wheel_left
- removed link wheel_right
- added link base_footprint
- added link lidar_link; collision mesh filename=package://omni_3w/meshes/omni_3w_lidar.obj scale=1 1 1; visual mesh filename=package://omni_3w/meshes/omni_3w_lidar.obj scale=1 1 1
- added link wheel_0; collision mesh filename=package://omni_3w/meshes/omni_3w_wheel_0.obj scale=1 1 1; visual mesh filename=package://omni_3w/meshes/omni_3w_wheel_0.obj scale=1 1 1
- added link wheel_1; collision mesh filename=package://omni_3w/meshes/omni_3w_wheel_1.obj scale=1 1 1; visual mesh filename=package://omni_3w/meshes/omni_3w_wheel_1.obj scale=1 1 1
- added link wheel_2; collision mesh filename=package://omni_3w/meshes/omni_3w_wheel_2.obj scale=1 1 1; visual mesh filename=package://omni_3w/meshes/omni_3w_wheel_2.obj scale=1 1 1
- link base_link: geometry collision mesh filename=package://omni_3w/meshes/omni_3w_chassis.obj scale=1 1 1; visual mesh filename=package://omni_3w/meshes/omni_3w_chassis.obj scale=1 1 1
Joints:
- added joint base_joint: type fixed, parent base_footprint, child base_link, origin xyz=0 0 0.07000 rpy=0 0 0
- added joint lidar_joint: type fixed, parent base_link, child lidar_link, origin xyz=0.00000 0.00000 0.07000 rpy=0 0 0
- added joint wheel_0_joint: type continuous, parent base_link, child wheel_0, origin xyz=0.12000 0.00000 -0.03000 rpy=0 0 0.00000, axis 0 1 0
- added joint wheel_1_joint: type continuous, parent base_link, child wheel_1, origin xyz=-0.06000 0.10400 -0.03000 rpy=0 0 2.09400, axis 0 1 0
- added joint wheel_2_joint: type continuous, parent base_link, child wheel_2, origin xyz=-0.06000 -0.10400 -0.03000 rpy=0 0 -2.09400, axis 0 1 0

File: packages/demos/simple_arm/urdf/robot.urdf (robot description, URDF)
Before this commit: robot simple_arm, 3 links, 0 joints
Links:
- removed link wheel_left
- removed link wheel_right
- added link base_footprint
- added link link1; collision mesh filename=package://simple_arm/meshes/simple_arm_link1.obj scale=1 1 1; visual mesh filename=package://simple_arm/meshes/simple_arm_link1.obj scale=1 1 1
- added link link2; collision mesh filename=package://simple_arm/meshes/simple_arm_link2.obj scale=1 1 1; visual mesh filename=package://simple_arm/meshes/simple_arm_link2.obj scale=1 1 1
- link base_link: geometry collision mesh filename=package://simple_arm/meshes/simple_arm_chassis.obj scale=1 1 1; visual mesh filename=package://simple_arm/meshes/simple_arm_chassis.obj scale=1 1 1
Joints:
- added joint base_joint: type fixed, parent base_footprint, child base_link, origin xyz=0 0 0.03000 rpy=0 0 0
- added joint link1_joint: type fixed, parent base_link, child link1, origin xyz=0.25000 0.00000 0.05000 rpy=0 0 0
- added joint link2_joint: type fixed, parent base_link, child link2, origin xyz=0.70000 0.00000 0.05000 rpy=0 0 0

File: packages/demos/tricycle_3w/urdf/robot.urdf (robot description, URDF)
Before this commit: robot tricycle_3w, 3 links, 0 joints
Links:
- removed link wheel_left
- removed link wheel_right
- added link base_footprint
- added link lidar_link; collision mesh filename=package://tricycle_3w/meshes/tricycle_3w_lidar.obj scale=1 1 1; visual mesh filename=package://tricycle_3w/meshes/tricycle_3w_lidar.obj scale=1 1 1
- added link wheel_rear_l; collision mesh filename=package://tricycle_3w/meshes/tricycle_3w_wheel_rear_l.obj scale=1 1 1; visual mesh filename=package://tricycle_3w/meshes/tricycle_3w_wheel_rear_l.obj scale=1 1 1
- added link wheel_rear_r; collision mesh filename=package://tricycle_3w/meshes/tricycle_3w_wheel_rear_r.obj scale=1 1 1; visual mesh filename=package://tricycle_3w/meshes/tricycle_3w_wheel_rear_r.obj scale=1 1 1
- added link wheel_steer; collision mesh filename=package://tricycle_3w/meshes/tricycle_3w_wheel_steer.obj scale=1 1 1; visual mesh filename=package://tricycle_3w/meshes/tricycle_3w_wheel_steer.obj scale=1 1 1
- link base_link: geometry collision mesh filename=package://tricycle_3w/meshes/tricycle_3w_chassis.obj scale=1 1 1; visual mesh filename=package://tricycle_3w/meshes/tricycle_3w_chassis.obj scale=1 1 1
Joints:
- added joint base_joint: type fixed, parent base_footprint, child base_link, origin xyz=0 0 0.08000 rpy=0 0 0
- added joint lidar_joint: type fixed, parent base_link, child lidar_link, origin xyz=0.08000 0.00000 0.07000 rpy=0 0 0
- added joint wheel_rear_l_joint: type continuous, parent base_link, child wheel_rear_l, origin xyz=-0.12000 0.12000 -0.03000 rpy=0 0 0.00000, axis 0 1 0
- added joint wheel_rear_r_joint: type continuous, parent base_link, child wheel_rear_r, origin xyz=-0.12000 -0.12000 -0.03000 rpy=0 0 0.00000, axis 0 1 0
- added joint wheel_steer_joint: type continuous, parent base_link, child wheel_steer, origin xyz=0.16000 0.00000 -0.03000 rpy=0 0 0.00000, axis 0 1 0
