Commit message: Improve product: upgrade cycle 2026-07-14d samples and tooling
- Add cycle sample/data/tooling improvement
- Bump patch version where applicable
- Keep ruff/pytest green

File: packages/demos/tricycle_3w/urdf/robot.urdf (robot description, URDF)
Before this commit: robot tricycle_3w, 6 links, 5 joints
Joints:
- joint base_joint: origin xyz=0 0 0.08000 rpy=0 0 0 -> xyz=0 0 0.14000 rpy=0 0 0
- joint lidar_joint: origin xyz=0.08000 0.00000 0.07000 rpy=0 0 0 -> xyz=0.00000 0.00000 0.16000 rpy=0 0 0
- joint wheel_rear_l_joint: origin xyz=-0.12000 0.12000 -0.03000 rpy=0 0 0.00000 -> xyz=-0.13000 0.15000 -0.04000 rpy=0 0 0.00000
- joint wheel_rear_r_joint: origin xyz=-0.12000 -0.12000 -0.03000 rpy=0 0 0.00000 -> xyz=-0.13000 -0.15000 -0.04000 rpy=0 0 0.00000
- joint wheel_steer_joint: origin xyz=0.16000 0.00000 -0.03000 rpy=0 0 0.00000 -> xyz=0.25000 0.00000 -0.05500 rpy=0 0 0.00000
